File: Displacement Sensor/Displacement Sensor.kicad_sch (KiCad schematic)
At the start: 16 parts, among them J1 DTF13-6P, U3 MCP2515-I, U4 TJA1050DRG, X1 ${ALTIUM_VALUE}

Commit message: Updated Labels
Parts:
- renumbered C11 to C1, C12 to C2, C13 to C3, C14 to C4, C15 to C5, R13 to R3, U4 to U1, U3 to U2
Changed lines of the file:
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@@
 		(on_board yes)
 		(dnp no)
-		(property "Reference" "C14"
+		(property "Reference" "C4"
 			(at 113.411 159.512 0)
 			(effects
@@
 			(project "Displacement Sensor"
 				(path "/f0211a9d-cfd7-4dfa-9b2f-9a363f96d705"
-					(reference "C14")
+					(reference "C4")
 					(unit 0)
 				)
@@
 		(on_board yes)
 		(dnp no)
-		(property "Reference" "C13"
+		(property "Reference" "C3"
 			(at 112.649 149.352 0)
 			(effects
@@
 			(project "Displacement Sensor"
 				(path "/f0211a9d-cfd7-4dfa-9b2f-9a363f96d705"
-					(reference "C13")
+					(reference "C3")
 					(unit 0)
 				)
@@
 		(on_board yes)
 		(dnp no)
-		(property "Reference" "C11"
+		(property "Reference" "C1"
 			(at 78.232 143.002 0)
 			(effects
@@
 			(project "Displacement Sensor"
 				(path "/f0211a9d-cfd7-4dfa-9b2f-9a363f96d705"
-					(reference "C11")
+					(reference "C1")
 					(unit 0)
 				)
@@
 		(on_board yes)
 		(dnp no)
-		(property "Reference" "U4"
+		(property "Reference" "U1"
 			(at 231.14 132.08 0)
 			(effects
@@
 			(project "Displacement Sensor"
 				(path "/f0211a9d-cfd7-4dfa-9b2f-9a363f96d705"
-					(reference "U4")
+					(reference "U1")
 					(unit 0)
 				)
@@
 		(on_board yes)
 		(dnp no)
-		(property "Reference" "C12"
+		(property "Reference" "C2"
 			(at 106.68 142.24 0)
 			(effects
@@
 			(project "Displacement Sensor"
 				(path "/f0211a9d-cfd7-4dfa-9b2f-9a363f96d705"
-					(reference "C12")
+					(reference "C2")
 					(unit 0)
 				)
@@
 		(on_board yes)
 		(dnp no)
-		(property "Reference" "U3"
+		(property "Reference" "U2"
 			(at 139.7 119.38 0)
 			(effects
@@
 			(project "Displacement Sensor"
 				(path "/f0211a9d-cfd7-4dfa-9b2f-9a363f96d705"
-					(reference "U3")
+					(reference "U2")
 					(unit 0)
 				)
@@
 		(on_board yes)
 		(dnp no)
-		(property "Reference" "C15"
+		(property "Reference" "C5"
 			(at 262.89 151.13 0)
 			(effects
@@
 			(project "Displacement Sensor"
 				(path "/f0211a9d-cfd7-4dfa-9b2f-9a363f96d705"
-					(reference "C15")
+					(reference "C5")
 					(unit 0)
 				)
@@
 		(dnp no)
 		(fields_autoplaced yes)
-		(property "Reference" "R13"
+		(property "Reference" "R3"
 			(at 125.73 130.81 90)
 			(effects
@@
 			(project "Displacement Sensor"
 				(path "/f0211a9d-cfd7-4dfa-9b2f-9a363f96d705"
-					(reference "R13")
+					(reference "R3")
 					(unit 1)
 				)
