File: New Tachometer/New Tachometer.kicad_pcb (KiCad board)
At the start: 2 copper layers, 54.8 x 71.2 mm, 35 parts, among them J1 DTF13-6P, Q1 NPN, U1 NE555P, U2 LM311, U3 MCP2515-I, U4 TJA1050DRG, X1 8MHz

Commit message: tachmeter
Parts:
- removed the REF** at (142.0, 130.5)
- removed the REF** at (142.0, 67.2)
- removed the REF** at (95.2, 130.5)
- removed the REF** at (95.2, 67.2)
- added G***: LOGO, Baja Logo:Baja Logo, B.Cu at (119.2, 82.3)
- added REF**: Fiducial_0.75mm_Mask1.5mm, Fiducial:Fiducial_0.75mm_Mask1.5mm, F.Cu at (99.0, 67.2)
- added REF**: Fiducial_0.75mm_Mask1.5mm, Fiducial:Fiducial_0.75mm_Mask1.5mm, F.Cu at (138.2, 130.7)
- added REF**: Fiducial_0.75mm_Mask1.5mm, Fiducial:Fiducial_0.75mm_Mask1.5mm, F.Cu at (138.3, 67.2)
- added REF**: Fiducial_0.75mm_Mask1.5mm, Fiducial:Fiducial_0.75mm_Mask1.5mm, F.Cu at (94.3, 126.8)
- J1: footprint 0_Baja_2025:TE_DTF13-6P -> New Tachometer:TE_DTF13-6P
- U1: renamed from U4; value TJA1050DRG -> NE555P; footprint Package_SO:SOIC-8_5.3x5.3mm_P1.27mm -> Package_DIP:DIP-8_W7.62mm
- U2: renamed from U3; value MCP2515-I -> LM311; footprint Package_SO:SOIC-18W_7.5x11.6mm_P1.27mm -> Package_DIP:DIP-8_W7.62mm
- U3: renamed from U2; value LM311 -> MCP2515-I; footprint Package_DIP:DIP-8_W7.62mm -> Package_SO:SOIC-18W_7.5x11.6mm_P1.27mm
- U4: renamed from U1; value NE555P -> TJA1050DRG; footprint Package_DIP:DIP-8_W7.62mm -> Package_SO:SOIC-8_5.3x5.3mm_P1.27mm
- moved U4 31.3 mm to (138.8, 95.2), turned to 0 degrees
- moved U2 31.1 mm to (117.7, 127.9)
- moved U3 30.9 mm to (108.2, 98.3)
- moved U1 29.7 mm to (113.8, 114.2), turned to 180 degrees
- moved J1 3.43 mm to (134.9, 112.2)
- moved C12 2.96 mm to (100.4, 128.4), turned to -90 degrees
- moved R1 2.40 mm to (127.9, 117.6)
- moved C4 2.23 mm to (115.3, 94.8)
- moved C3 1.45 mm to (132.2, 96.8)
- moved C13 1.32 mm to (101.7, 123.8), turned to 180 degrees
- moved D2 1.20 mm to (123.7, 110.2)
- moved C5 0.78 mm to (141.0, 91.5)
- moved D1 0.30 mm to (118.7, 110.2)
- moved Q1 0.20 mm to (124.9, 102.3)
- moved R13 0.10 mm to (118.1, 105.1)
- renumbered C11 to C1, C1 to C11, C2 to C12, C3 to C13, C4 to C14, C12 to C2, C13 to C3, C14 to C4, C15 to C5, R3 to R13, R13 to R3
Connections:
- R13 pad 1: +5v -> +5V
- R9 pad 1: +5v -> +5V
- U1 pad 1: Net-(U3-TXCAN) -> GND
- U1 pad 2: GND -> 555 input
- U1 pad 3: +5V -> 555 output
- U1 pad 4: Net-(U3-RXCAN) -> +5V
- U1 pad 5: unconnected-(U4-SPLIT-Pad5) -> Net-(U1-CV)
- U1 pad 6: Low -> Net-(U1-DIS)
- U1 pad 7: High -> Net-(U1-DIS)
- U1 pad 8: GND -> +5V
- U2 pad 1: Net-(U3-TXCAN) -> GND
- U2 pad 2: Net-(U3-RXCAN) -> Net-(U2-+)
- U2 pad 3: unconnected-(U3-CLKOUT/SOF-Pad3) -> Comparator input
- U2 pad 4: unconnected-(U3-~{TX0RTS}-Pad4) -> GND
- U2 pad 7: Net-(U3-OSC2) -> 555 input
- U2 pad 8: Net-(U3-OSC1) -> +5V
- U3 pad 1: GND -> Net-(U3-TXCAN)
- U3 pad 2: Net-(U2-+) -> Net-(U3-RXCAN)
- U3 pad 3: Comparator input -> unconnected-(U3-CLKOUT/SOF-Pad3)
- U3 pad 4: GND -> unconnected-(U3-~{TX0RTS}-Pad4)
- U3 pad 7: 555 input -> Net-(U3-OSC2)
- U3 pad 8: +5v -> Net-(U3-OSC1)
- U4 pad 1: GND -> Net-(U3-TXCAN)
- U4 pad 2: 555 input -> GND
- U4 pad 3: 555 output -> +5V
- U4 pad 4: +5V -> Net-(U3-RXCAN)
- U4 pad 5: Net-(U1-CV) -> unconnected-(U4-SPLIT-Pad5)
- U4 pad 6: Net-(U1-DIS) -> Low
- U4 pad 7: Net-(U1-DIS) -> High
- U4 pad 8: +5V -> GND
Routing:
- net +5v: track 39.7 -> 0.00 mm
- net +5V: track 143.2 -> 182.7 mm
- net Net-(U3-OSC2): track 31.7 -> 38.4 mm
- net arduino input: track 83.6 -> 87.5 mm
- net Net-(U3-TXCAN): track 37.1 -> 39.9 mm
- net Net-(D1-K): track 9.77 -> 12.4 mm
- net Net-(U3-RXCAN): track 37.4 -> 39.8 mm
- net GND: track 25.1 -> 22.6 mm
- net Net-(U3-OSC1): track 15.7 -> 17.9 mm
- net Comparator input: track 33.2 -> 35.4 mm
- net Low: track 26.6 -> 25.2 mm
- net Net-(U3-~{RESET}): track 6.15 -> 7.37 mm
- net High: track 30.2 -> 29.1 mm
- net SO: track 31.2 -> 30.6 mm
- net CS: track 27.4 -> 26.9 mm
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Other:
- outline, holes or cut-outs redrawn

Commit message: tach
Parts:
- removed the REF** at (99.0, 67.2)
- removed the REF** at (138.2, 130.7)
- removed the REF** at (138.3, 67.2)
- removed the REF** at (94.3, 126.8)
- added REF**: Fiducial_0.75mm_Mask1.5mm, Fiducial:Fiducial_0.75mm_Mask1.5mm, F.Cu at (94.5, 126.3)
- added REF**: Fiducial_0.75mm_Mask1.5mm, Fiducial:Fiducial_0.75mm_Mask1.5mm, F.Cu at (137.8, 131.1)
- added REF**: Fiducial_0.75mm_Mask1.5mm, Fiducial:Fiducial_0.75mm_Mask1.5mm, F.Cu at (99.2, 67.3)
- added REF**: Fiducial_0.75mm_Mask1.5mm, Fiducial:Fiducial_0.75mm_Mask1.5mm, F.Cu at (138.1, 67.2)
- moved U4 1.25 mm to (113.8, 115.4)
- moved R10 1.15 mm to (113.9, 125.9)
- moved R4 1.15 mm to (113.9, 121.4)
- moved R6 1.15 mm to (106.2, 119.2)
- moved R7 1.15 mm to (106.2, 123.7)
- moved R8 1.15 mm to (106.2, 128.2)
- moved R9 1.15 mm to (106.2, 130.4)
- moved U2 0.50 mm to (108.2, 98.8)
- renumbered U4 to U1, U3 to U2, U2 to U3, U1 to U4
Connections:
- U2 pad 12: unconnected-(U3-~{INT}-Pad12) -> Net-(U2-~{INT})
- UNIT_1 pad 12: INT -> unconnected-(UNIT_1-D9-Pad12)
- UNIT_1 pad 5: unconnected-(UNIT_1-D2-Pad5) -> Net-(U2-~{INT})
Routing:
- net Net-(U2-~{INT}): track 0.00 -> 12.0 mm, vias 0 -> 1
- net +5V: track 182.7 -> 173.6 mm
- net 555 output: track 22.5 -> 30.0 mm, vias 0 -> 2
- net GND: track 22.6 -> 18.5 mm
- net Net-(U4-CV): track 12.5 -> 14.1 mm
- net Net-(U2-OSC2): track 38.4 -> 39.8 mm
- net Net-(U2-OSC1): track 17.9 -> 19.1 mm
- net 555 input: track 19.7 -> 20.5 mm
- net Net-(U1-RXD): track 39.8 -> 40.6 mm
- net Net-(U3-+): track 10.2 -> 9.69 mm
