File: New Tachometer/New Tachometer.kicad_sch (KiCad schematic)
At the start: 31 parts, among them J1 DTF13-6P, Q1 NPN, U1 NE555P, U2 LM311, U3 MCP2515-I, U4 TJA1050DRG, X1 ${ALTIUM_VALUE}

Commit message: tachmeter
Parts:
- J1: footprint 0_Baja_2025:TE_DTF13-6P -> New Tachometer:TE_DTF13-6P
- renumbered C11 to C1, C1 to C11, C2 to C12, C3 to C13, C4 to C14, C12 to C2, C13 to C3, C14 to C4, C15 to C5, R3 to R13, R13 to R3
Connections:
- net +5v is gone; now on net VCC: R13.1, R9.1, U2.8 (V+)
Changed lines of the file:
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@@
 	(wire
 		(pts
+			(xy 127 119.38) (xy 127 121.92)
+		)
+		(stroke
+			(width 0)
+			(type default)
+		)
+	)
+	(wire
+		(pts
 			(xy 293.37 129.54) (xy 322.58 129.54)
 		)
@@
 	(wire
 		(pts
+			(xy 241.3 36.83) (xy 238.76 36.83)
+		)
+		(stroke
+			(width 0)
+			(type default)
+		)
+	)
+	(wire
+		(pts
 			(xy 34.29 50.8) (xy 36.83 50.8)
 		)
@@
 		)
 	)
-	(global_label "+5v"
+	(global_label "+5V"
 		(shape input)
 		(at 124.46 20.32 90)
@@
 		)
 		(property "Intersheetrefs" "${INTERSHEET_REFS}"
-			(at 124.46 13.5853 90)
+			(at 124.46 13.4643 90)
 			(effects
 				(font
@@
 	(global_label "INT"
 		(shape input)
-		(at 127 121.92 90)
+		(at 127 119.38 90)
 		(fields_autoplaced yes)
 		(effects
@@
 		)
 		(property "Intersheetrefs" "${INTERSHEET_REFS}"
-			(at 127 116.0319 90)
+			(at 127 113.4919 90)
 			(effects
 				(font
@@
 	(global_label "+5V"
 		(shape input)
-		(at 238.76 36.83 0)
+		(at 241.3 36.83 0)
 		(fields_autoplaced yes)
 		(effects
@@
 		)
 		(property "Intersheetrefs" "${INTERSHEET_REFS}"
-			(at 245.6157 36.83 0)
+			(at 248.1557 36.83 0)
 			(effects
 				(font
@@
 		)
 	)
-	(global_label "+5v"
+	(global_label "+5V"
 		(shape input)
 		(at 67.31 66.04 180)
@@
 		)
 		(property "Intersheetrefs" "${INTERSHEET_REFS}"
-			(at 60.5753 66.04 0)
+			(at 60.4543 66.04 0)
 			(effects
 				(font
@@
 		)
 	)
-	(global_label "+5v"
+	(global_label "+5V"
 		(shape input)
 		(at 107.95 68.58 90)
@@
 		)
 		(property "Intersheetrefs" "${INTERSHEET_REFS}"
-			(at 107.95 61.8453 90)
+			(at 107.95 61.7243 90)
 			(effects
 				(font
@@
 			)
 		)
-		(property "Footprint" "0_Baja_2025:TE_DTF13-6P"
+		(property "Footprint" "New Tachometer:TE_DTF13-6P"
 			(at 46.99 53.34 0)
 			(effects
@@
 		(dnp no)
 		(fields_autoplaced yes)
-		(property "Reference" "C1"
+		(property "Reference" "C11"
 			(at 215.9 89.2809 0)
 			(effects
@@
 			(project "New Tachometer"
 				(path "/5984495b-0ee4-4b65-b298-d000695921f9"
-					(reference "C1")
+					(reference "C11")
 					(unit 1)
 				)
@@
 		(dnp no)
 		(fields_autoplaced yes)
-		(property "Reference" "C2"
+		(property "Reference" "C12"
 			(at 233.68 89.2809 0)
 			(effects
@@
 			(project "New Tachometer"
 				(path "/5984495b-0ee4-4b65-b298-d000695921f9"
-					(reference "C2")
+					(reference "C12")
 					(unit 1)
 				)
@@
 		(on_board yes)
 		(dnp no)
-		(property "Reference" "C14"
+		(property "Reference" "C4"
 			(at 209.931 154.432 0)
 			(effects
@@
 			(project "New Tachometer"
 				(path "/5984495b-0ee4-4b65-b298-d000695921f9"
-					(reference "C14")
+					(reference "C4")
 					(unit 0)
 				)
@@
 		(on_board yes)
 		(dnp no)
-		(property "Reference" "C13"
+		(property "Reference" "C3"
 			(at 209.169 144.272 0)
 			(effects
@@
 			(project "New Tachometer"
 				(path "/5984495b-0ee4-4b65-b298-d000695921f9"
-					(reference "C13")
+					(reference "C3")
 					(unit 0)
 				)
@@
 		(on_board yes)
 		(dnp no)
-		(property "Reference" "C11"
+		(property "Reference" "C1"
 			(at 174.752 137.922 0)
 			(effects
@@
 			(project "New Tachometer"
 				(path "/5984495b-0ee4-4b65-b298-d000695921f9"
-					(reference "C11")
+					(reference "C1")
 					(unit 0)
 				)
@@
 		(on_board yes)
 		(dnp no)
-		(property "Reference" "C4"
+		(property "Reference" "C14"
 			(at 207.264 26.162 0)
 			(effects
@@
 			(project "New Tachometer"
 				(path "/5984495b-0ee4-4b65-b298-d000695921f9"
-					(reference "C4")
+					(reference "C14")
 					(unit 1)
 				)
@@
 		(dnp no)
 		(property "Reference" "U4"
-			(at 327.66 127 0)
+			(at 327.406 127 0)
 			(effects
 				(font
@@
 		(on_board yes)
 		(dnp no)
-		(property "Reference" "C12"
+		(property "Reference" "C2"
 			(at 203.2 137.16 0)
 			(effects
@@
 			(project "New Tachometer"
 				(path "/5984495b-0ee4-4b65-b298-d000695921f9"
-					(reference "C12")
+					(reference "C2")
 					(unit 0)
 				)
@@
 		(dnp no)
 		(fields_autoplaced yes)
-		(property "Reference" "C3"
+		(property "Reference" "C13"
 			(at 221.869 63.5 90)
 			(effects
@@
 			(project "New Tachometer"
 				(path "/5984495b-0ee4-4b65-b298-d000695921f9"
-					(reference "C3")
+					(reference "C13")
 					(unit 1)
 				)
@@
 		(on_board yes)
 		(dnp no)
-		(property "Reference" "C15"
+		(property "Reference" "C5"
 			(at 359.41 146.05 0)
 			(effects
@@
 			(project "New Tachometer"
 				(path "/5984495b-0ee4-4b65-b298-d000695921f9"
-					(reference "C15")
+					(reference "C5")
 					(unit 0)
 				)
@@
 		(dnp no)
 		(fields_autoplaced yes)
-		(property "Reference" "R13"
+		(property "Reference" "R3"
 			(at 222.25 125.73 90)
 			(effects
@@
 			(project "New Tachometer"
 				(path "/5984495b-0ee4-4b65-b298-d000695921f9"
-					(reference "R13")
+					(reference "R3")
 					(unit 1)
 				)
@@
 		(dnp no)
 		(fields_autoplaced yes)
-		(property "Reference" "R3"
+		(property "Reference" "R13"
 			(at 127 22.8599 0)
 			(effects
@@
 			(project "New Tachometer"
 				(path "/5984495b-0ee4-4b65-b298-d000695921f9"
-					(reference "R3")
+					(reference "R13")
 					(unit 1)
 				)

Commit message: tach
Parts:
- renumbered U4 to U1, U3 to U2, U2 to U3, U1 to U4
Connections:
- net INT: no longer names the net of UNIT_1.12 (D9)
- no-connect marks 28 -> 27
Changed lines of the file:
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@@
 	)
 	(no_connect
+		(at 127 121.92)
+	)
+	(no_connect
 		(at 129.54 157.48)
 	)
@@
 	)
 	(no_connect
-		(at 269.24 139.7)
-	)
-	(no_connect
 		(at 104.14 157.48)
 	)
@@
 	)
 	(no_connect
-		(at 127 157.48)
-	)
-	(no_connect
 		(at 124.46 121.92)
 	)
@@
 	(wire
 		(pts
-			(xy 127 119.38) (xy 127 121.92)
-		)
-		(stroke
-			(width 0)
-			(type default)
-		)
-	)
-	(wire
-		(pts
 			(xy 293.37 129.54) (xy 322.58 129.54)
 		)
@@
 	(wire
 		(pts
+			(xy 269.24 139.7) (xy 278.13 139.7)
+		)
+		(stroke
+			(width 0)
+			(type default)
+		)
+	)
+	(wire
+		(pts
 			(xy 212.09 87.63) (xy 218.44 87.63)
 		)
@@
 	(wire
 		(pts
+			(xy 127 171.45) (xy 127 157.48)
+		)
+		(stroke
+			(width 0)
+			(type default)
+		)
+	)
+	(wire
+		(pts
 			(xy 207.01 154.94) (xy 207.01 157.48)
 		)
@@
 	(wire
 		(pts
+			(xy 278.13 171.45) (xy 127 171.45)
+		)
+		(stroke
+			(width 0)
+			(type default)
+		)
+	)
+	(wire
+		(pts
 			(xy 81.28 35.56) (xy 87.63 35.56)
 		)
@@
 	(wire
 		(pts
+			(xy 278.13 139.7) (xy 278.13 171.45)
+		)
+		(stroke
+			(width 0)
+			(type default)
+		)
+	)
+	(wire
+		(pts
 			(xy 111.76 160.02) (xy 111.76 157.48)
 		)
@@
 		)
 	)
-	(global_label "INT"
-		(shape input)
-		(at 127 119.38 90)
-		(fields_autoplaced yes)
-		(effects
-			(font
-				(size 1.27 1.27)
-			)
-			(justify left)
-		)
-		(property "Intersheetrefs" "${INTERSHEET_REFS}"
-			(at 127 113.4919 90)
-			(effects
-				(font
-					(size 1.27 1.27)
-				)
-				(justify left)
-				(hide yes)
-			)
-		)
-	)
 	(global_label "arduino input"
 		(shape input)
@@
 		(on_board yes)
 		(dnp no)
-		(property "Reference" "U4"
+		(property "Reference" "U1"
 			(at 327.406 127 0)
 			(effects
@@
 			(project "New Tachometer"
 				(path "/5984495b-0ee4-4b65-b298-d000695921f9"
-					(reference "U4")
+					(reference "U1")
 					(unit 0)
 				)
@@
 		(on_board yes)
 		(dnp no)
-		(property "Reference" "U3"
+		(property "Reference" "U2"
 			(at 236.22 114.3 0)
 			(effects
@@
 			(project "New Tachometer"
 				(path "/5984495b-0ee4-4b65-b298-d000695921f9"
-					(reference "U3")
+					(reference "U2")
 					(unit 0)
 				)
@@
 		(on_board yes)
 		(dnp no)
-		(property "Reference" "U2"
+		(property "Reference" "U3"
 			(at 124.46 69.8814 0)
 			(effects
@@
 			(project "New Tachometer"
 				(path "/5984495b-0ee4-4b65-b298-d000695921f9"
-					(reference "U2")
+					(reference "U3")
 					(unit 1)
 				)
@@
 		(dnp no)
 		(fields_autoplaced yes)
-		(property "Reference" "U1"
-			(at 241.3 30.5114 90)
+		(property "Reference" "U4"
+			(at 241.3 30.4098 90)
 			(effects
 				(font
@@
 		)
 		(property "Value" "NE555P"
-			(at 241.3 33.0514 90)
+			(at 241.3 32.9498 90)
 			(effects
 				(font
@@
 			(project "New Tachometer"
 				(path "/5984495b-0ee4-4b65-b298-d000695921f9"
-					(reference "U1")
+					(reference "U4")
 					(unit 1)
 				)
