File: Main Computer/Main Computer.kicad_sch (KiCad schematic)
At the start: 6 parts, among them J1 Pi 5 GPIO HEADER, J2 Conn_01x06, J3 Conn_01x02, J4 CAN to outer connector, U1 RFM9X Breakout

Commit message: Revert PCB (footprint nonsense)
This reverts commit 10dbf7cf734bf138f5810b545ad3c613d1decc14.
Connections:
- net SCK: now also UNIT_1.2 (SCK)
- net SI: now also UNIT_1.3 (SI)
- net SO: now also UNIT_1.4 (SO)
- net INT: now reaches J1.22 (GPIO_25)
- net INT: now also UNIT_1.1 (INT)
- net CS: now reaches J1.24 (GPIO_8)
- net CS: now also UNIT_1.5 (CS)
- net CAN_CS: no longer names the net of J1.36 (GPIO_16)
- net CAN_CS: no longer UNIT_1.5 (CS)
- net CAN_INT: no longer names the net of J1.15 (GPIO_22)
- net CAN_INT: no longer UNIT_1.1 (INT)
- net SPI1_MISO: no longer names the net of J1.35 (GPIO_19)
- net SPI1_MISO: no longer UNIT_1.4 (SO)
- net SPI1_MOSI: no longer names the net of J1.38 (GPIO_20)
- net SPI1_MOSI: no longer UNIT_1.3 (SI)
- net SPI1_SCK: no longer names the net of J1.40 (GPIO_21)
- net SPI1_SCK: no longer UNIT_1.2 (SCK)
- no-connect marks 26 -> 8
