File: Main Computer/Main Computer.kicad_pcb (KiCad board)
At the start: 2 copper layers, 56 x 65 mm, 11 parts, among them J1 Pi 5 GPIO HEADER, J3 Conn_01x02, J4 CAN to outer connector, U1 RFM9X Breakout

Commit message: Rev 2, DRC pass
Other:
- board text added: "MAIN COMPUTER '26 REV 2"
- board text removed: "MAIN COMPUTER '26 REV 1"
Changed lines of the file:
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@@
 		(effects
 			(font
-				(size 1.1 1.1)
+				(size 1.2 1.2)
 				(thickness 0.1)
 			)
@@
 		)
 	)
-	(gr_text "MAIN COMPUTER '26\nREV 1\n"
+	(gr_text "MAIN COMPUTER '26\nREV 2\n"
 		(at 143.1 148 90)
 		(layer "F.SilkS")
@@
 	)
 	(segment
-		(start 145.685 113.25)
-		(end 131 113.25)
+		(start 146.25 112.685)
+		(end 145.935 113)
 		(width 0.5)
 		(layer "F.Cu")
@@
 	)
 	(segment
-		(start 146.25 112.685)
-		(end 145.685 113.25)
+		(start 145.935 113)
+		(end 131.25 113)
 		(width 0.5)
 		(layer "F.Cu")
@@
 	)
 	(segment
-		(start 131 113.25)
+		(start 131.25 113)
 		(end 127.76 116.49)
 		(width 0.5)
